Commit message: fixed the transition to the frontier + fixed integration with reactive planner

File: urdf/iris/iris_with_sensors.xacro (robot description, xacro)
@@ -122,15 +122,17 @@
   <xacro:include filename="$(find victim_localization)/urdf/iris_accessories/realsense_camera.urdf.xacro"/>
  <xacro:realsense_camera name="front_cam" parent="base_link">
-    <origin xyz="0 0 -0.048" rpy="0 0.26179 0"/> <!--15 deg for pitch -->
+    <origin xyz="0 0 -0.05" rpy="0 0.26179 0"/> <!--15 deg for pitch -->
   </xacro:realsense_camera>
   <!-- Thermal Facing RGB camera -->
+ <!--
    <xacro:include filename="$(find victim_localization)/urdf/iris_accessories/generic_camera.urdf.xacro" />
     <xacro:generic_camera name="thermal_cam" parent="base_link" ros_topic="RGB/image_raw" cam_info_topic="RGB/camera_info" update_rate="77" res_x="1228" res_y="1027" image_format="R8G8B8" hfov="52.9855">
-    <origin xyz="0.0 0.0 -0.05" rpy="0 0.26179 0"/>  <!--15 deg for pitch -->
+    <origin xyz="0.0 0.0 -0.05" rpy="0 0.26179 0"/>
   </xacro:generic_camera>
  <xacro:include filename="$(find victim_localization)/urdf/iris_accessories/generic_thermal_camera.urdf.xacro" />
   <xacro:generic_thermal_camera name="thermal_cam" parent="base_link" ros_topic="thermal/image_raw" cam_info_topic="RGB/camera_info" update_rate="10" res_x="160" res_y="120" image_format="R8G8B8" hfov="52.9855">
-  <origin xyz="0.0 0.0 -0.05" rpy="0 0.26179 0"/>  <!--15 deg for pitch -->
+  <origin xyz="0.0 0.0 -0.05" rpy="0 0.26179 0"/>
 </xacro:generic_thermal_camera>
+-->
   <!-- stick -->
       <!-- Spawn velodyne -->

File: urdf/iris/iris_with_sensors_kuri.urdf (robot description, URDF)
Before this commit: robot iris, 14 links, 13 joints
Links:
- added link downward_cam_link, mass 0.001; collision box size=0.01 0.01 0.01; visual box size=0.01 0.01 0.01
- added link downward_cam_optical_frame
Joints:
- added joint downward_cam_joint: type fixed, parent base_link, child downward_cam_link, origin xyz=0.0 0.0 -0.045 rpy=0 1.57079632679 0
- added joint downward_cam_optical_joint: type fixed, parent downward_cam_link, child downward_cam_optical_frame, origin xyz=0 0 0 rpy=-1.57079632679 0.0 -1.57079632679
- joint front_cam_joint: origin xyz=0 0 -0.05 rpy=0 0.26179 0 -> xyz=0 0 -0.048 rpy=0 0 0
