Commit message: added settings file + changes to combined map

File: urdf/iris/iris_with_sensors.urdf (robot description, URDF)
Before this commit: robot iris, 16 links, 15 joints
Links:
- removed link downward_cam_link
- removed link downward_cam_optical_frame
- added link thermal_cam_link, mass 0.001; collision box size=0.01 0.01 0.01; visual box size=0.01 0.01 0.01
- added link thermal_cam_optical_frame
- added link thermal_cam_thermal_link, mass 0.001; collision box size=0.01 0.01 0.01; visual box size=0.01 0.01 0.01
- added link thermal_cam_thermal_optical_frame
Joints:
- removed joint downward_cam_joint
- removed joint downward_cam_optical_joint
- added joint thermal_cam_joint: type fixed, parent base_link, child thermal_cam_link, origin xyz=0.0 0.0 -0.06 rpy=0 0.26179 0
- added joint thermal_cam_optical_joint: type fixed, parent thermal_cam_link, child thermal_cam_optical_frame, origin xyz=0 0 0 rpy=-1.57079632679 0.0 -1.57079632679
- added joint thermal_cam_thermal_joint: type fixed, parent base_link, child thermal_cam_thermal_link, origin xyz=0.0 0.0 -0.06 rpy=0 0.26179 0
- added joint thermal_cam_thermal_optical_joint: type fixed, parent thermal_cam_thermal_link, child thermal_cam_thermal_optical_frame, origin xyz=0 0 0 rpy=-1.57079632679 0.0 -1.57079632679

File: urdf/iris/iris_with_sensors.xacro (robot description, xacro)
@@ -122,20 +122,15 @@
   <xacro:include filename="$(find victim_localization)/urdf/iris_accessories/realsense_camera.urdf.xacro"/>
  <xacro:realsense_camera name="front_cam" parent="base_link">
-    <origin xyz="0 0 -0.048" rpy="0 0.26179 0"/> <!--previous 0.093 for pitch -->
+    <origin xyz="0 0 -0.048" rpy="0 0.26179 0"/> <!--15 deg for pitch -->
   </xacro:realsense_camera>
-  <!-- forward facing thermal camera -->
-<!--
-    <xacro:include filename="$(find victim_localization)/urdf/iris_accessories/flir_a35_camera.urdf.xacro"/>
- <xacro:flir_a35_camera name="front_cam" parent="base_link">
-    <origin xyz="0.15 0 -0.048" rpy="0 0.093 0"/>
-  </xacro:flir_a35_camera>
--->
-  <!-- Downward facing camera -->
+  <!-- Thermal Facing RGB camera -->
    <xacro:include filename="$(find victim_localization)/urdf/iris_accessories/generic_camera.urdf.xacro" />
- <!-- <xacro:generic_camera name="downward_cam" parent="base_link" ros_topic="camera/image" cam_info_topic="camera/camera_info" update_rate="20" res_x="640" res_y="480" image_format="R8G8B8" hfov="100">
-    <origin xyz="0.0 0.0 -0.045" rpy="0 ${M_PI/2} 0"/> -->
-    <xacro:generic_camera name="downward_cam" parent="base_link" ros_topic="camera/image" cam_info_topic="camera/camera_info" update_rate="77" res_x="1228" res_y="1027" image_format="R8G8B8" hfov="52.9855">
-    <origin xyz="0.0 0.0 -0.045" rpy="0 ${M_PI/2} 0"/>  <!-- previous ${M_PI/2} -->
+    <xacro:generic_camera name="thermal_cam" parent="base_link" ros_topic="RGB/image_raw" cam_info_topic="RGB/camera_info" update_rate="77" res_x="1228" res_y="1027" image_format="R8G8B8" hfov="52.9855">
+    <origin xyz="0.0 0.0 -0.06" rpy="0 0.26179 0"/>  <!--15 deg for pitch -->
   </xacro:generic_camera>
+ <xacro:include filename="$(find victim_localization)/urdf/iris_accessories/generic_thermal_camera.urdf.xacro" />
+  <xacro:generic_thermal_camera name="thermal_cam" parent="base_link" ros_topic="thermal/image_raw" cam_info_topic="RGB/camera_info" update_rate="10" res_x="160" res_y="120" image_format="R8G8B8" hfov="52.9855">
+  <origin xyz="0.0 0.0 -0.06" rpy="0 0.26179 0"/>  <!--15 deg for pitch -->
+</xacro:generic_thermal_camera>
   <!-- stick -->
       <!-- Spawn velodyne -->

Commit message: added rosinstall and navigation test node

File: urdf/iris/iris_with_sensors.urdf (robot description, URDF)
Before this commit: robot iris, 18 links, 17 joints
Joints:
- joint thermal_cam_joint: origin xyz=0.0 0.0 -0.06 rpy=0 0.26179 0 -> xyz=0.0 0.0 -0.05 rpy=0 0.26179 0
- joint thermal_cam_thermal_joint: origin xyz=0.0 0.0 -0.06 rpy=0 0.26179 0 -> xyz=0.0 0.0 -0.05 rpy=0 0.26179 0

File: urdf/iris/iris_with_sensors.xacro (robot description, xacro)
@@ -127,9 +127,9 @@
    <xacro:include filename="$(find victim_localization)/urdf/iris_accessories/generic_camera.urdf.xacro" />
     <xacro:generic_camera name="thermal_cam" parent="base_link" ros_topic="RGB/image_raw" cam_info_topic="RGB/camera_info" update_rate="77" res_x="1228" res_y="1027" image_format="R8G8B8" hfov="52.9855">
-    <origin xyz="0.0 0.0 -0.06" rpy="0 0.26179 0"/>  <!--15 deg for pitch -->
+    <origin xyz="0.0 0.0 -0.05" rpy="0 0.26179 0"/>  <!--15 deg for pitch -->
   </xacro:generic_camera>
  <xacro:include filename="$(find victim_localization)/urdf/iris_accessories/generic_thermal_camera.urdf.xacro" />
   <xacro:generic_thermal_camera name="thermal_cam" parent="base_link" ros_topic="thermal/image_raw" cam_info_topic="RGB/camera_info" update_rate="10" res_x="160" res_y="120" image_format="R8G8B8" hfov="52.9855">
-  <origin xyz="0.0 0.0 -0.06" rpy="0 0.26179 0"/>  <!--15 deg for pitch -->
+  <origin xyz="0.0 0.0 -0.05" rpy="0 0.26179 0"/>  <!--15 deg for pitch -->
 </xacro:generic_thermal_camera>
   <!-- stick -->

Commit message: Raytacing is fast now, Viewpoint evaluation take 1s for 1 iteration compared to previously 12s + code clean up

File: urdf/iris/iris_with_sensors.urdf (robot description, URDF)
Before this commit: robot iris, 14 links, 13 joints
Links:
- link front_cam_link: mass 0.000200 -> 0.000000
Joints:
- joint front_cam_joint: origin xyz=0 0 -0.05 rpy=0 0.26179 0 -> xyz=0 0 0.07 rpy=0 0 0

File: urdf/iris/iris_with_sensors.xacro (robot description, xacro)
@@ -122,17 +122,7 @@
   <xacro:include filename="$(find victim_localization)/urdf/iris_accessories/realsense_camera.urdf.xacro"/>
  <xacro:realsense_camera name="front_cam" parent="base_link">
-    <origin xyz="0 0 -0.05" rpy="0 0.26179 0"/> <!--15 deg for pitch -->
+    <origin xyz="0.0 0.0 -0.05" rpy="0 0.26179 0"/> <!--15 deg for pitch -->  <!-- previous "0.0 0.0 -0.05" rpy="0 0.26179 0"/> -->
   </xacro:realsense_camera>
   <!-- Thermal Facing RGB camera -->
- <!--
-   <xacro:include filename="$(find victim_localization)/urdf/iris_accessories/generic_camera.urdf.xacro" />
-    <xacro:generic_camera name="thermal_cam" parent="base_link" ros_topic="RGB/image_raw" cam_info_topic="RGB/camera_info" update_rate="77" res_x="1228" res_y="1027" image_format="R8G8B8" hfov="52.9855">
-    <origin xyz="0.0 0.0 -0.05" rpy="0 0.26179 0"/>
-  </xacro:generic_camera>
- <xacro:include filename="$(find victim_localization)/urdf/iris_accessories/generic_thermal_camera.urdf.xacro" />
-  <xacro:generic_thermal_camera name="thermal_cam" parent="base_link" ros_topic="thermal/image_raw" cam_info_topic="RGB/camera_info" update_rate="10" res_x="160" res_y="120" image_format="R8G8B8" hfov="52.9855">
-  <origin xyz="0.0 0.0 -0.05" rpy="0 0.26179 0"/>
-</xacro:generic_thermal_camera>
--->
   <!-- stick -->
       <!-- Spawn velodyne -->

File: urdf/iris_accessories/generic_camera.urdf.xacro (robot description, xacro)
@@ -10,7 +10,7 @@
     <link name="${name}_link">
       <inertial>
-        <mass value="0.001" />
+        <mass value="0.000" />
         <origin xyz="0 0 0" rpy="0 0 0" />
-        <inertia ixx="0.0001" ixy="0" ixz="0" iyy="0.0001" iyz="0" izz="0.0001" />
+        <inertia ixx="0.0000" ixy="0" ixz="0" iyy="0.0000" iyz="0" izz="0.0000" />
       </inertial>
       <visual>

File: urdf/iris_accessories/generic_thermal_camera.urdf.xacro (robot description, xacro)
@@ -10,7 +10,7 @@
     <link name="${name}_thermal_link">
       <inertial>
-        <mass value="0.001" />
+        <mass value="0.000" />
         <origin xyz="0 0 0" rpy="0 0 0" />
-        <inertia ixx="0.0001" ixy="0" ixz="0" iyy="0.0001" iyz="0" izz="0.0001" />
+        <inertia ixx="0.0000" ixy="0" ixz="0" iyy="0.0000" iyz="0" izz="0.0000" />
       </inertial>
       <visual>

File: urdf/iris_accessories/realsense_camera.urdf.xacro (robot description, xacro)
@@ -14,7 +14,7 @@
       <link name="${name}_link">
         <inertial>
-          <mass value="0.000200" />
+          <mass value="0.000000" />
           <origin xyz="0 0 0" rpy="0 0 0" />
-          <inertia ixx="5.8083e-4" ixy="0" ixz="0" iyy="3.0833e-5" iyz="0" izz="5.9083e-4" />
+          <inertia ixx="0" ixy="0" ixz="0" iyy="0" iyz="0" izz="0" />
         </inertial>
         <visual>

Commit message: last update

File: urdf/iris/iris_with_sensors.urdf (robot description, URDF)
Before this commit: robot iris, 14 links, 13 joints
Links:
- added link thermal_cam_link, mass 0.000; collision box size=0.01 0.01 0.01; visual box size=0.01 0.01 0.01
- added link thermal_cam_optical_frame
- added link thermal_cam_thermal_link, mass 0.000; collision box size=0.01 0.01 0.01; visual box size=0.01 0.01 0.01
- added link thermal_cam_thermal_optical_frame
Joints:
- added joint thermal_cam_joint: type fixed, parent base_link, child thermal_cam_link, origin xyz=0.0 0.0 -0.05 rpy=0 0.26179 0
- added joint thermal_cam_optical_joint: type fixed, parent thermal_cam_link, child thermal_cam_optical_frame, origin xyz=0 0 0 rpy=-1.57079632679 0.0 -1.57079632679
- added joint thermal_cam_thermal_joint: type fixed, parent base_link, child thermal_cam_thermal_link, origin xyz=0.0 0.0 -0.05 rpy=0 0.26179 0
- added joint thermal_cam_thermal_optical_joint: type fixed, parent thermal_cam_thermal_link, child thermal_cam_thermal_optical_frame, origin xyz=0 0 0 rpy=-1.57079632679 0.0 -1.57079632679
- joint front_cam_joint: origin xyz=0 0 0.07 rpy=0 0 0 -> xyz=0.0 0.0 -0.05 rpy=0 0.26179 0

File: urdf/iris/iris_with_sensors.xacro (robot description, xacro)
@@ -125,4 +125,13 @@
   </xacro:realsense_camera>
   <!-- Thermal Facing RGB camera -->
+  <!-- Thermal Facing RGB camera -->
+   <xacro:include filename="$(find victim_localization)/urdf/iris_accessories/generic_camera.urdf.xacro" />
+    <xacro:generic_camera name="thermal_cam" parent="base_link" ros_topic="RGB/image_raw" cam_info_topic="RGB/camera_info" update_rate="77" res_x="1228" res_y="1027" image_format="R8G8B8" hfov="52.9855">
+    <origin xyz="0.0 0.0 -0.05" rpy="0 0.26179 0"/>
+  </xacro:generic_camera>
+ <xacro:include filename="$(find victim_localization)/urdf/iris_accessories/generic_thermal_camera.urdf.xacro" />
+  <xacro:generic_thermal_camera name="thermal_cam" parent="base_link" ros_topic="thermal/image_raw" cam_info_topic="RGB/camera_info" update_rate="10" res_x="160" res_y="120" image_format="R8G8B8" hfov="52.9855">
+  <origin xyz="0.0 0.0 -0.05" rpy="0 0.26179 0"/>
+</xacro:generic_thermal_camera>
   <!-- stick -->
       <!-- Spawn velodyne -->
